File: Hardware/ESP-V.kicad_pcb (KiCad board)
At the start: 2 copper layers, 56 parts, among them J1 USB_C_Receptacle_USB2.0, J2 Conn_01x16_Male, J3 Conn_01x14_Female, J4 Conn_Coaxial, U1 AT25xxx-MA, U2 AP7333-33SRG-7, U3 AP7333-33SRG-7, U4 ESP32-C3, U5 CH552G, Y1 40MHz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

Commit message: Update ESP-V.kicad_pcb
Parts:
- moved C15 14.7 mm to (130.6, 121.0)
- moved C18 13.1 mm to (129.8, 110.2)
- moved C16 5.64 mm to (110.9, 118.9), turned to 315 degrees
- moved C13 5.26 mm to (110.0, 119.8), turned to 315 degrees
- moved C24 2.26 mm to (111.9, 117.9)
- moved C11 1.35 mm to (113.5, 117.1), turned to 315 degrees
- moved C19 0.37 mm to (109.0, 120.8)
Routing:
- net +3V3: track 4.49 -> 32.4 mm, vias 0 -> 2
- net /GP00: track 1.18 -> 11.1 mm
- net /GP03: track 1.04 -> 8.49 mm
- net /GP01: track 4.09 -> 10.9 mm
- net /GP04: track 0.00 -> 6.74 mm
- net /LEDTX: track 0.00 -> 6.63 mm
- net /ESP_ENABLE: track 1.99 -> 7.27 mm, vias 0 -> 2
- net /GP02: track 3.40 -> 8.33 mm
- net /LEDRX: track 0.00 -> 4.18 mm
- net /GP07: track 0.00 -> 3.87 mm
- net /GP06: track 0.00 -> 3.13 mm
- net Net-(D2-Pad1): track 0.00 -> 2.01 mm
- net Net-(D3-Pad1): track 0.00 -> 1.99 mm
- net /GP05: track 0.00 -> 1.65 mm
- net GND: vias 0 -> 10
Other:
- net class Default: via_dia 0.8 -> 0.65
- net class power added: clearance 0.5, trace_width 0.4, via_dia 1, via_drill 0.6
- net class thin added: clearance 0.15, trace_width 0.15, via_dia 0.65, via_drill 0.35
- rule trace_min: 0.2 -> 0.15
- rule via_min_drill: 0.3 -> 0.35
- rule via_min_size: 0.4 -> 0.65

Commit message: Update ESP-V.kicad_pcb
Parts:
- removed TP3: t1, TestPoint:TestPoint_Pad_D4.0mm
- removed TP4: t2, TestPoint:TestPoint_Pad_D4.0mm
- removed TP5: t3, TestPoint:TestPoint_Pad_D4.0mm
- removed TP6: t4, TestPoint:TestPoint_Pad_D4.0mm
- C15, C18: moved to B.Cu
- moved J2 40.2 mm to (116.3, 119.2)
- moved C20 35.2 mm to (102.6, 105.7), turned to 135 degrees
- moved C18 30.1 mm to (127.9, 140.2)
- moved J3 28.2 mm to (90.8, 81.2)
- moved C14 27.7 mm to (109.8, 108.6)
- moved C23 27.3 mm to (109.4, 110.2)
- moved C17 25.9 mm to (103.6, 104.7), turned to 135 degrees
- moved C15 16.7 mm to (132.3, 137.6)
- moved C25 7.93 mm to (94.5, 99.4), turned to 90 degrees
- moved C26 6.93 mm to (94.5, 96.0), turned to 270 degrees
- moved C12 6.57 mm to (111.0, 105.0), turned to 90 degrees
- moved RN1 5.45 mm to (107.7, 105.0)
- moved D2 4.51 mm to (108.4, 95.5)
- moved D3 4.51 mm to (108.4, 101.0)
- moved R3 4.51 mm to (108.2, 97.3)
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Routing:
- net +3.3VA: track 8.57 -> 47.4 mm, vias 2 -> 4
- net /GP10: track 3.76 -> 31.1 mm, vias 0 -> 1
- net VDD: track 0.00 -> 27.3 mm
- net /BLSEL: track 5.49 -> 28.8 mm, vias 0 -> 1
- net /GP08: track 5.63 -> 27.1 mm, vias 0 -> 1
- net +3V3: track 32.4 -> 52.5 mm
- net /GP05: track 1.65 -> 21.2 mm
- net /GP07: track 3.87 -> 22.7 mm, vias 0 -> 1
- net /CHUSB-: track 0.00 -> 18.3 mm, vias 0 -> 1
- net /CHUSB+: track 2.43 -> 20.5 mm
- net /GP06: track 3.13 -> 20.7 mm, vias 0 -> 1
- net /ESP_ENABLE: track 7.27 -> 22.8 mm
- net VBUS: track 0.00 -> 15.5 mm, vias 0 -> 2
- net /GP04: track 6.74 -> 19.5 mm
- net /CC2: track 0.00 -> 10.5 mm
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
Commit message: finished routing + front silk
Parts:
- added G***: LOGO, art and silk:frontsilk, F.Cu at (99.7, 97.3)
- J4: footprint Connector_Coaxial:SMA_Amphenol_132289_EdgeMount -> footprint:ACAG0801-2450-T
- moved Y2 44.4 mm to (111.6, 118.7)
- moved C15 26.2 mm to (111.6, 121.5), turned to 270 degrees
- moved C18 23.8 mm to (113.2, 121.5), turned to 270 degrees
- moved J4 22.9 mm to (89.5, 123.0), turned to 0 degrees
- moved C10 9.35 mm to (91.3, 116.2), turned to 180 degrees
- moved C21 5.80 mm to (101.5, 120.5)
- moved C9 5.30 mm to (91.3, 114.8), turned to 180 degrees
- moved C22 4.92 mm to (101.5, 124.0)
- moved Y1 4.34 mm to (94.8, 115.0), turned to 0 degrees
- moved L2 2.39 mm to (101.4, 122.3), turned to 180 degrees
- moved J2 2.30 mm to (116.2, 116.8)
- moved J3 2.30 mm to (90.7, 78.8)
- moved C26 0.55 mm to (95.1, 96.0)
- moved C25 0.55 mm to (95.1, 99.4)
- moved C1 0.55 mm to (96.0, 80.0)
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Connections:
- J1 pad 1: (no net) -> GND
- J4 pad 2: GND -> (no net)
Routing:
- net +3V3: track 52.5 -> 117.7 mm, vias 2 -> 3
- net /ESPUSB-: track 2.53 -> 55.1 mm
- net /ESPUSB+: track 3.17 -> 48.4 mm
- net VBUS: track 15.5 -> 53.8 mm, vias 2 -> 3
- net /ESP_RX: track 3.72 -> 34.1 mm, vias 0 -> 2
- net /GP11: track 8.04 -> 37.3 mm
- net /ESP_TX: track 4.53 -> 32.6 mm, vias 1 -> 2
- net /GP13: track 9.64 -> 30.3 mm, vias 2 -> 3
- net /GP12: track 14.5 -> 34.1 mm, vias 1 -> 2
- net /GP01: track 15.7 -> 34.7 mm, vias 0 -> 2
- net /GP14: track 11.5 -> 29.0 mm
- net /GP15: track 10.5 -> 25.9 mm, vias 1 -> 2
- net /GP00: track 15.1 -> 29.7 mm, vias 0 -> 2
- net /GP16: track 10.3 -> 23.6 mm, vias 1 -> 2
- net /GP17: track 13.5 -> 26.1 mm, vias 1 -> 0
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- added copper zone on B.Cu, net GND
- added copper zone on F.Cu, net GND
Other:
- board outline added: 29.1 x 48.2 mm
- net class rf added: clearance 0.4, trace_width 0.4, via_dia 0.65, via_drill 0.35

Commit message: ready to order needs final check
Parts:
- added G***: LOGO, art and silk:backsilk, B.Cu at (102.3, 100.8)
- Y2: footprint Crystal:Crystal_DS10_D1.0mm_L4.3mm_Horizontal -> footprint:Crystal_DS10_D1.0mm_L4.3mm_Horizontalnosilk
- turned C5 to 0 degrees
Connections:
- J2 pad 1: +3V3 -> GND
- J2 pad 15: GND -> +3.3VA
- J2 pad 16: GND -> +3V3
- J2 pad 2: +3.3VA -> GND
Routing:
- net +3.3VA: track 52.2 -> 66.0 mm
- net +3V3: track 117.7 -> 124.3 mm, vias 3 -> 4
- net VBUS: track 53.8 -> 51.7 mm
- net /GP17: track 26.1 -> 25.3 mm
- net GND: track 3.02 -> 3.57 mm, vias 81 -> 80
Other:
- board text added: "V1.0"
