File: Hardware/DEBUG.sch (KiCad schematic (older format))
At the start: 6 parts, among them U5 CH552G

Commit message: redesigning to take module
Parts:
- removed U5: CH552G, Housings_SOIC:SOIC-16_3.9x9.9mm_Pitch1.27mm, symbol MCU_WCH:CH552G
- added U1: CH552E, Package_SO:MSOP-10_3x3mm_P0.5mm, symbol MCU_WCH:CH552E
Connections:
- net labels removed: CHP11, CHP14, CHP15, CHP16, CHP17, CHP33, CHRESET, P11, P14, P15, P16, P17, P33
- wire segments 46 -> 34
Changed lines of the file:
@@
 EESchema Schematic File Version 4
-LIBS:MeshangerV-cache
+LIBS:ESP-V-cache
 EELAYER 26 0
 EELAYER END
 $Descr A4 11693 8268
 encoding utf-8
-Sheet 3 3
+Sheet 2 2
 Title ""
 Date ""
@@
 3V3
 $Comp
-L MCU_WCH:CH552G U5
-U 1 1 5FDED1AF
-P 7200 3600
-F 0 "U5" H 7175 4315 50  0000 C CNN
-F 1 "CH552G" H 7175 4224 50  0000 C CNN
-F 2 "Housings_SOIC:SOIC-16_3.9x9.9mm_Pitch1.27mm" H 7500 3600 50  0001 C CNN
-F 3 "" H 7500 3600 50  0001 C CNN
-	1    7200 3600
-	1    0    0    -1
-$EndComp
-$Comp
 L power:VBUS #PWR?
 U 1 1 5FDEDEFB
@@
 $EndComp
 Wire Wire Line
-	8400 3600 9000 3600
-Wire Wire Line
-	8400 3750 9000 3750
-Wire Wire Line
-	5950 4050 5500 4050
-Wire Wire Line
-	5950 4200 5500 4200
+	8400 3800 9000 3800
+Wire Wire Line
+	8400 3950 9000 3950
+Wire Wire Line
+	5950 3800 5500 3800
+Wire Wire Line
+	5950 3950 5500 3950
 Wire Wire Line
 	5950 3150 5500 3150
 Wire Wire Line
 	5500 3150 5500 2800
-$Comp
-L power:VBUS #PWR?
-U 1 1 5FDF0272
-P 5500 2800
-AR Path="/5FDF0272" Ref="#PWR?"  Part="1"
-AR Path="/5FDE49AF/5FDF0272" Ref="#PWR?"  Part="1"
-AR Path="/5FF3EE03/5FDF0272" Ref="#PWR041"  Part="1"
-F 0 "#PWR041" H 5500 2650 50  0001 C CNN
-F 1 "VBUS" H 5515 2973 50  0000 C CNN
-F 2 "" H 5500 2800 50  0001 C CNN
-F 3 "" H 5500 2800 50  0001 C CNN
-	1    5500 2800
-	1    0    0    -1
-$EndComp
 Wire Wire Line
 	8400 3450 9000 3450
@@
 Wire Wire Line
 	8700 3150 8700 2800
-Wire Wire Line
-	5950 3300 5500 3300
-Text Label 5500 4050 0    50   ~ 0
+Text Label 5500 3800 0    50   ~ 0
 DEBUGRX
-Text Label 5500 4200 0    50   ~ 0
+Text Label 5500 3950 0    50   ~ 0
 DEBUGTX
 Wire Wire Line
-	5950 3450 5500 3450
-Wire Wire Line
-	5950 3600 5500 3600
-Wire Wire Line
-	5950 3750 5500 3750
-Wire Wire Line
-	5950 3900 5500 3900
-Wire Wire Line
-	8400 3900 9000 3900
-Wire Wire Line
-	8400 4050 9000 4050
-Wire Wire Line
-	8400 4200 9000 4200
-Text Label 9000 3600 0    50   ~ 0
+	5950 3650 5500 3650
+Text Label 9000 3800 0    50   ~ 0
 USB-
-Text Label 9000 3750 0    50   ~ 0
+Text Label 9000 3950 0    50   ~ 0
 USB+
 Wire Wire Line
@@
 Text Label 2200 900  0    50   ~ 0
 GND
-Text Label 5500 3900 0    50   ~ 0
-CHRESET
-Text Label 5500 3750 0    50   ~ 0
-P17
-Text Label 5500 3600 0    50   ~ 0
-P16
-Text Label 9000 4200 0    50   ~ 0
-P11
-Text Label 5500 3450 0    50   ~ 0
-P15
-Text Label 5500 3300 0    50   ~ 0
-P14
-Text Label 9000 3900 0    50   ~ 0
+Text Label 5500 3500 0    50   ~ 0
 ESPRESET
 Text Label 4900 900  0    50   ~ 0
@@
 Wire Wire Line
 	3650 700  3800 700
-Text HLabel 4500 600  0    50   Input ~ 0
-CHP11
 Text HLabel 4500 700  0    50   Input ~ 0
 ESP_BL
@@
 DEBUGRX
 Wire Wire Line
-	4900 600  4500 600
-Wire Wire Line
 	4500 700  4900 700
 Wire Wire Line
@@
 Wire Wire Line
 	4900 1000 4500 1000
-Text HLabel 5650 700  0    50   Input ~ 0
-CHP15
-Text HLabel 5650 600  0    50   Input ~ 0
-CHP14
-Text HLabel 5650 800  0    50   Input ~ 0
-CHP16
-Text HLabel 5650 900  0    50   Input ~ 0
-CHP17
-Wire Wire Line
-	5650 600  5950 600
-Wire Wire Line
-	5950 700  5650 700
-Wire Wire Line
-	5650 800  5950 800
-Wire Wire Line
-	5950 900  5650 900
 Wire Wire Line
 	9250 5000 9600 5000
@@
 	1    0    0    -1
 $EndComp
-Text Label 9000 4050 0    50   ~ 0
-P33
-Text Label 5950 600  0    50   ~ 0
-P14
-Text Label 5950 700  0    50   ~ 0
-P15
-Text Label 5950 800  0    50   ~ 0
-P16
-Text Label 5950 900  0    50   ~ 0
-P17
-Text Label 5950 1000 0    50   ~ 0
-P33
-Text Label 4900 600  0    50   ~ 0
-P11
-Text HLabel 5650 1000 0    50   Input ~ 0
-CHP33
-Wire Wire Line
-	5950 1000 5650 1000
 $Comp
 L Device:C_Small C25
@@
 Text Label 7050 2600 0    50   ~ 0
 GND
+$Comp
+L MCU_WCH:CH552E U1
+U 1 1 5FE7DAF8
+P 7200 3550
+F 0 "U1" H 7175 4215 50  0000 C CNN
+F 1 "CH552E" H 7175 4124 50  0000 C CNN
+F 2 "Package_SO:MSOP-10_3x3mm_P0.5mm" H 7050 2850 50  0001 C CNN
+F 3 "" H 7500 3500 50  0001 C CNN
+	1    7200 3550
+	1    0    0    -1
+$EndComp
+Wire Wire Line
+	5500 3500 5950 3500
+Text Label 5500 3650 0    50   ~ 0
+ESPBL
+Text Label 5500 2800 0    50   ~ 0
+3V3
 $EndSCHEMATC
