File: Hardware/antenna.sch (KiCad schematic (older format))
At the start: 4 parts, among them J4 Conn_Coaxial

Commit message: Update antenna.sch
Parts:
- renumbered C22 to C?, C21 to C?, J4 to J?, L2 to L?
Changed lines of the file:
@@
 EESchema Schematic File Version 4
-LIBS:MeshangerV-cache
-EELAYER 26 0
+LIBS:ESP-V-cache
+EELAYER 29 0
 EELAYER END
 $Descr A4 11693 8268
 encoding utf-8
-Sheet 4 3
+Sheet 4 2
 Title ""
 Date ""
@@
 VCC
 $Comp
-L Device:L_Small L2
+L Device:L_Small L?
 U 1 1 5FC5BF06
 P 4400 3200
-F 0 "L2" H 4447 3246 50  0000 L CNN
+F 0 "L?" H 4447 3246 50  0000 L CNN
 F 1 "L_Small" H 4447 3155 50  0000 L CNN
 F 2 "Inductor_SMD:L_0603_1608Metric" H 4400 3200 50  0001 C CNN
@@
 $EndComp
 $Comp
-L Device:C_Small C22
+L Device:C_Small C?
 U 1 1 5FC5BFAB
 P 4950 3550
-F 0 "C22" H 5042 3596 50  0000 L CNN
+F 0 "C?" H 5042 3596 50  0000 L CNN
 F 1 "C_Small" H 5042 3505 50  0000 L CNN
 F 2 "Capacitors_SMD:C_0603_HandSoldering" H 4950 3550 50  0001 C CNN
@@
 $EndComp
 $Comp
-L Device:C_Small C21
+L Device:C_Small C?
 U 1 1 5FC5C01F
 P 3750 3550
-F 0 "C21" H 3842 3596 50  0000 L CNN
+F 0 "C?" H 3842 3596 50  0000 L CNN
 F 1 "C_Small" H 3842 3505 50  0000 L CNN
 F 2 "Capacitors_SMD:C_0603_HandSoldering" H 3750 3550 50  0001 C CNN
@@
 	4950 3650 4950 4100
 $Comp
-L Connector:Conn_Coaxial J4
+L Connector:Conn_Coaxial J?
 U 1 1 5FC624A8
 P 5500 3200
-F 0 "J4" H 5600 3175 50  0000 L CNN
+F 0 "J?" H 5600 3175 50  0000 L CNN
 F 1 "Conn_Coaxial" H 5600 3084 50  0000 L CNN
 F 2 "Connector_Coaxial:SMA_Amphenol_132289_EdgeMount" H 5500 3200 50  0001 C CNN
