File: Hardware/ESP-V.sch (KiCad schematic (older format))
At the start: 46 parts, among them J1 USB_C_Receptacle_USB2.0, J2 Conn_01x16_Male, J3 Conn_01x14_Female, U1 AT25xxx-MA, U2 AP7333-33SRG-7, U3 AP7333-33SRG-7, U4 ESP32-C3, Y1 40MHz, Y2 32k

Commit message: redesigning to take module
Parts:
- removed C10, C9: 10nF, Capacitors_SMD:C_0603_HandSoldering, symbol Device:C_Small
- removed C6: 100nF, Capacitors_SMD:C_0603_HandSoldering, symbol Device:C_Small
- removed D2, D3: LED_ALT, LED_SMD:LED_0805_2012Metric_Pad1.15x1.40mm_HandSolder, symbol Device:LED_ALT
- removed J2: Conn_01x16_Male, Connector_PinHeader_2.54mm:PinHeader_1x16_P2.54mm_Vertical, symbol Connector:Conn_01x16_Male
- removed R3, R4: 1k, Resistor_SMD:R_0603_1608Metric_Pad1.05x0.95mm_HandSolder, symbol Device:R_Small
- removed TP3: t1, TestPoint:TestPoint_Pad_D4.0mm, symbol Connector:TestPoint
- removed TP4: t2, TestPoint:TestPoint_Pad_D4.0mm, symbol Connector:TestPoint
- removed TP5: t3, TestPoint:TestPoint_Pad_D4.0mm, symbol Connector:TestPoint
- removed TP6: t4, TestPoint:TestPoint_Pad_D4.0mm, symbol Connector:TestPoint
- removed U1: AT25xxx-MA, Package_DFN_QFN:DFN-8-1EP_3x2mm_P0.5mm_EP1.75x1.45mm, symbol Memory_EEPROM:AT25xxx-MA
- removed Y1: 40MHz, Crystal:Crystal_SMD_Abracon_ABM10-4Pin_2.5x2.0mm, symbol Device:Crystal_GND24
- added J2: Conn_01x14_Female, Connector_PinHeader_2.54mm:PinHeader_1x14_P2.54mm_Vertical, symbol Connector:Conn_01x14_Female
- added J4: USB_A, Connectors:USB_A, symbol Connector:USB_A
Connections:
- net labels removed: LEDRX, LEDTX, TOUCH0, TOUCH1, TOUCH2, TOUCH3
- wire segments 266 -> 222
Other:
- note added: "USBA port for host mode\n"
- note added: "defaults to using ESPUSB for prog and debug\n"
- note removed: "COMMS LEDS\n"

Commit message: v1.1 ready to order
Parts:
- removed C1: 100uF, Capacitors_SMD:CP_Elec_4x4.5, symbol Device:CP
- removed C11, C12: 22uF 0805, Capacitors_SMD:C_0805_HandSoldering, symbol Device:C_Small
- removed C13, C3, C5, C8: 1uF, Capacitors_SMD:C_0603_HandSoldering, symbol Device:C_Small
- removed C14, C2: 10uF, Capacitors_SMD:C_0805_HandSoldering, symbol Device:C_Small
- removed C15, C18: 10nF, Capacitors_SMD:C_0603_HandSoldering, symbol Device:C_Small
- removed C16: 100nF, Capacitors_SMD:C_0603_HandSoldering, symbol Device:C_Small
- removed C17: 10uF, Capacitors_SMD:C_0603_HandSoldering, symbol Device:C_Small
- removed C19: 10pF, Capacitors_SMD:C_0603_HandSoldering, symbol Device:C_Small
- removed C24: 100nF, Capacitor_SMD:C_0603_1608Metric_Pad1.05x0.95mm_HandSolder, symbol Device:C_Small
- removed J2, J3: Conn_01x14_Female, Connector_PinHeader_2.54mm:PinHeader_1x14_P2.54mm_Vertical, symbol Connector:Conn_01x14_Female
- removed U2, U3: AP7333-33SRG-7, TO_SOT_Packages_SMD:SOT-23, symbol Diodes_inc:AP7333-33SRG-7
- removed U4: ESP32-C3, Package_DFN_QFN:QFN-32-1EP_5x5mm_P0.5mm_EP3.45x3.45mm, symbol ESP-V-rescue:ESP32-C3-MCU_Espressif-MeshangerV-rescue
- removed Y2: 32k, Crystal:Crystal_DS10_D1.0mm_L4.3mm_Horizontal, symbol Device:Crystal
- added D2: LED, LED_SMD:LED_0603_1608Metric_Castellated, symbol Device:LED
- added J2, J3: Conn_01x10_Female, Connector_PinSocket_2.54mm:PinSocket_1x10_P2.54mm_Vertical, symbol Connector:Conn_01x10_Female
- added R3: R_Small, Resistor_SMD:R_0603_1608Metric_Pad1.05x0.95mm_HandSolder, symbol Device:R_Small
- added U2: NCP1117-3.3_SOT223, Package_TO_SOT_SMD:SOT-223-3_TabPin2, symbol Regulator_Linear:NCP1117-3.3_SOT223
- added U3: ESP32-C3-MINI-1, footprint:ESP32-c3-mini1, symbol Useful_ICs:ESP32-C3-MINI-1
- C20: value 1uF -> 10uF; footprint Capacitors_SMD:C_0603_HandSoldering -> Capacitor_SMD:C_0805_2012Metric_Pad1.15x1.40mm_HandSolder
- D1: footprint Diode_SMD:D_1210_3225Metric -> Diode_SMD:D_SOD-323
- L1: footprint Inductor_SMD:L_1210_3225Metric -> Inductor_SMD:L_0805_2012Metric_Pad1.15x1.40mm_HandSolder
Connections:
- net labels removed: +3.3VA, ANT, GP11, GP12, GP13, GP14, GP15, GP16, GP17, SPICS0, SPID, SPIHD, SPIQ, SPISCK, SPIWP, SPI_VCC
- wire segments 222 -> 142
Other:
- note removed: "Bulk caps to allow battery to take over"
- note removed: "optional \n"
